File: PCB/YukiBoard/YukiBoard.kicad_pcb (KiCad board)
At the start: 2 copper layers, 137.4 x 89.5 mm, 61 parts, among them J1 Conn_01x02, J2 Conn_01x02, SW1 SW_Push_45deg, SW10 SW_Push_45deg, SW11 SW_Push_45deg, SW12 SW_Push_45deg, SW13 SW_Push_45deg, SW14 SW_Push_45deg, SW15 SW_Push_45deg, SW16 SW_Push_45deg, SW17 SW_Push_45deg, SW18 SW_Push_45deg, SW19 SW_Push_45deg, SW2 SW_Push_45deg, SW20 SW_Push_45deg, SW21 SW_Push_45deg, SW22 SW_Push_45deg, SW23 SW_Push_45deg, SW24 SW_Push_45deg, SW25 SW_Push_45deg, SW26 SW_Push_45deg, SW27 SW_Push_45deg, SW28 SW_Push_45deg, SW29 SW_Push_45deg, SW3 SW_Push_45deg, SW30 SW_Push_45deg, SW31 SW_Push_45deg, SW32 SW_Push_45deg, SW33 SW_Push_45deg, SW34 SW_Push_45deg, SW35 SW_Push_45deg, SW36 SW_Push_45deg, SW37 SW_Push_45deg, SW38 SW_Push_45deg, SW39 SW_SPDT, SW4 SW_Push_45deg, SW5 SW_Push_45deg, SW6 SW_Push_45deg, SW7 SW_Push_45deg, SW8 SW_Push_45deg, SW9 SW_Push_45deg, U1 XIAO-nRF52840-DIP

Commit message: Add cool stuff to pcb 󰇳
Parts:
- moved SW15 30.4 mm to (101.2, 65.8)
- moved SW18 30.4 mm to (113.5, 88.0)
- moved SW23 30.4 mm to (101.2, 27.7)
- moved SW28 30.4 mm to (101.2, 46.7)
- moved SW34 30.4 mm to (101.2, 65.8)
- moved SW37 30.4 mm to (113.5, 88.0)
- moved SW4 30.4 mm to (101.2, 27.7)
- moved SW9 30.4 mm to (101.2, 46.7)
- moved SW13 30.4 mm to (62.6, 63.9)
- moved SW2 30.4 mm to (60.6, 25.8)
- moved SW21 30.4 mm to (60.6, 25.8)
- moved SW32 30.4 mm to (62.6, 63.9)
- moved SW11 30.4 mm to (23.4, 61.2)
- moved SW30 30.4 mm to (23.4, 61.2)
- moved D1 30.4 mm to (132.5, 61.2)
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Other:
- board text added: "3"
- board text added: ":"
- board text added: "Diodes 󰱫"
- board text added: "Keys"
- board text added: "Made wi"
- board text added: "Made with  by"
- board text added: "Rever"
- board text added: "manni"
- board text added: "sible 󰌌"
- board text added: "th  by manni"
- board text added: "󰬽"
- board text added: "󰭁"

Commit message: Add stuf
Parts:
- added D20: D, Diode_SMD:D_SOD-123, F.Cu at (175.8, 29.8)
- added D21: D, Diode_SMD:D_SOD-123, F.Cu at (178.1, 29.8)
- added D22: D, Diode_SMD:D_SOD-123, F.Cu at (180.4, 29.8)
- added D23: D, Diode_SMD:D_SOD-123, F.Cu at (175.8, 34.5)
- added D24: D, Diode_SMD:D_SOD-123, F.Cu at (178.1, 34.5)
- added D25: D, Diode_SMD:D_SOD-123, F.Cu at (180.4, 34.5)
- added D26: D, Diode_SMD:D_SOD-123, F.Cu at (175.8, 39.2)
- added D27: D, Diode_SMD:D_SOD-123, F.Cu at (178.1, 39.2)
- added D28: D, Diode_SMD:D_SOD-123, F.Cu at (180.4, 39.2)
- added D29: D, Diode_SMD:D_SOD-123, F.Cu at (175.8, 43.9)
- added D30: D, Diode_SMD:D_SOD-123, F.Cu at (178.1, 43.9)
- added D31: D, Diode_SMD:D_SOD-123, F.Cu at (180.4, 43.9)
- added D32: D, Diode_SMD:D_SOD-123, F.Cu at (175.8, 53.3)
- added D33: D, Diode_SMD:D_SOD-123, F.Cu at (175.8, 48.6)
- added D34: D, Diode_SMD:D_SOD-123, F.Cu at (178.1, 48.6)
- added D35: D, Diode_SMD:D_SOD-123, F.Cu at (180.4, 48.6)
- added D36: D, Diode_SMD:D_SOD-123, F.Cu at (178.1, 53.3)
- added D37: D, Diode_SMD:D_SOD-123, F.Cu at (180.4, 53.3)
- added D38: D, Diode_SMD:D_SOD-123, F.Cu at (176.4, 85.0)
- added REF**: mousebites 2mm, PCM_marbastlib-various:mousebites_2.5mm, F.Cu at (172.7, 74.8)
- added REF**: mousebites 2mm, PCM_marbastlib-various:mousebites_2.5mm, F.Cu at (172.7, 29.9)
- added REF**: mousebites 2mm, PCM_marbastlib-various:mousebites_2.5mm, B.Cu at (141.5, 74.8)
- added REF**: mousebites 2mm, PCM_marbastlib-various:mousebites_2.5mm, B.Cu at (141.4, 29.9)
- added SW40: SW_SPDT, ScottoKeebs_Components:Switch_MSK12C02, F.Cu at (258.9, 16.9)
- added U2: Seeeduino Xiao nRF52840, PCM_marbastlib-xp-promicroish:Xiao_nRF52840_ACH, F.Cu at (277.6, 26.1)
- SW1, SW10, SW11, SW12, SW13, SW14, SW15, SW16, SW17, SW18, SW19, SW2, SW3, SW4, SW5, SW6, SW7, SW8, SW9: moved to B.Cu
- U1: value XIAO-nRF52840-DIP -> Seeeduino Xiao nRF52840; footprint XIAO-:XIAO-nRF52840-DIP -> PCM_marbastlib-xp-promicroish:Xiao_nRF52840_ACH
- moved SW30 266.8 mm to (290.1, 68.6), turned to 169 degrees
- moved SW20 235.6 mm to (275.0, 46.3), turned to 169 degrees
- moved SW25 230.3 mm to (271.4, 65.0), turned to 169 degrees
- moved SW31 225.0 mm to (267.7, 83.7), turned to 169 degrees
- moved SW21 193.0 mm to (253.5, 28.7), turned to 174 degrees
- moved SW26 190.0 mm to (251.5, 47.6), turned to 174 degrees
- moved SW32 187.0 mm to (249.5, 66.6), turned to 174 degrees
- moved SW22 147.4 mm to (229.5, 22.7)
- moved SW27 147.4 mm to (229.5, 41.7)
- moved SW33 147.4 mm to (229.5, 60.8)
- moved J2 117.8 mm to (252.7, 81.3), turned to 0 degrees
- moved SW36 116.5 mm to (209.2, 90.7)
- moved SW28 109.3 mm to (210.4, 46.5)
- moved SW34 109.3 mm to (210.4, 65.5)
- moved SW23 109.3 mm to (210.4, 27.4)
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Connections:
- J1 pad 1: Net-(J1-Pin_1) -> /BAT-
- J2 pad 1: Net-(J2-Pin_1) -> /BAT-L
- J2 pad 2: Net-(J1-Pin_1) -> Net-(J2-Pin_2)
- SW20 pad 1: /C0 -> /C0L
- SW20 pad 2: Net-(D1-A) -> Net-(D20-A)
- SW21 pad 1: /C1 -> /C1L
- SW21 pad 2: Net-(D2-A) -> Net-(D21-A)
- SW22 pad 1: /C2 -> /C2L
- SW22 pad 2: Net-(D3-A) -> Net-(D22-A)
- SW23 pad 1: /C3 -> /C3L
- SW23 pad 2: Net-(D4-A) -> Net-(D23-A)
- SW24 pad 1: /C4 -> /C4L
- SW24 pad 2: Net-(D5-A) -> Net-(D24-A)
- SW25 pad 1: /C0 -> /C0L
- SW25 pad 2: Net-(D6-A) -> Net-(D25-A)
- SW26 pad 1: /C1 -> /C1L
- SW26 pad 2: Net-(D7-A) -> Net-(D26-A)
- SW27 pad 1: /C2 -> /C2L
- SW27 pad 2: Net-(D8-A) -> Net-(D27-A)
- SW28 pad 1: /C3 -> /C3L
- SW28 pad 2: Net-(D9-A) -> Net-(D28-A)
- SW29 pad 1: /C4 -> /C4L
- SW29 pad 2: Net-(D10-A) -> Net-(D29-A)
- SW30 pad 1: /C0 -> /C0L
- SW30 pad 2: Net-(D11-A) -> Net-(D30-A)
- SW31 pad 1: /C0 -> /C0L
- SW31 pad 2: Net-(D12-A) -> Net-(D31-A)
- SW32 pad 1: /C1 -> /C1L
- SW32 pad 2: Net-(D13-A) -> Net-(D32-A)
- SW33 pad 1: /C2 -> /C2L
- SW33 pad 2: Net-(D14-A) -> Net-(D33-A)
- SW34 pad 1: /C3 -> /C3L
- SW34 pad 2: Net-(D15-A) -> Net-(D34-A)
- SW35 pad 1: /C4 -> /C4L
- SW35 pad 2: Net-(D16-A) -> Net-(D35-A)
- SW36 pad 1: /C2 -> /C2L
- SW36 pad 2: Net-(D17-A) -> Net-(D36-A)
- SW37 pad 1: /C3 -> /C3L
- SW37 pad 2: Net-(D18-A) -> Net-(D37-A)
- SW38 pad 1: /C4 -> /C4L
- SW38 pad 2: Net-(D19-A) -> Net-(D38-A)
- SW39 pad 3: Net-(J2-Pin_1) -> /BAT+
- U1 pad 10: /R1 -> +3V3
- U1 pad 12: +3V3 -> /R1
- U1 pad 13: GND -> /R2
- U1 pad 14: VBUS -> /R3
- U1 pad 8: /R3 -> VBUS
- U1 pad 9: /R2 -> GND
Routing:
- net /C4L: track 0.00 -> 197.1 mm, vias 0 -> 1
- net /R2: track 52.7 -> 243.3 mm, vias 3 -> 1
- net /C0: track 259.2 -> 74.6 mm, vias 4 -> 0
- net /C3L: track 0.00 -> 172.2 mm, vias 0 -> 4
- net /R3L: track 0.00 -> 145.7 mm, vias 0 -> 6
- net /C2L: track 0.00 -> 143.7 mm, vias 0 -> 2
- net /R3: track 17.7 -> 154.3 mm, vias 1 -> 6
- net Net-(D30-A): track 0.00 -> 131.3 mm, vias 0 -> 3
- net Net-(D31-A): track 0.00 -> 130.0 mm, vias 0 -> 3
- net /R2L: track 0.00 -> 117.1 mm, vias 0 -> 4
- net /R1L: track 0.00 -> 116.2 mm, vias 0 -> 4
- net Net-(D20-A): track 0.00 -> 115.0 mm, vias 0 -> 1
- net /R0L: track 0.00 -> 114.5 mm, vias 0 -> 4
- net Net-(D32-A): track 0.00 -> 114.3 mm, vias 0 -> 1
- net /C0L: track 0.00 -> 113.4 mm
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- added copper zone on B.Cu, net GND
- added copper zone on F.Cu, net GND
- added copper zone on B.Cu, net GNDL
- added copper zone on F.Cu, net GNDL
Other:
- board size 137.4 x 89.5 mm -> 288.1 x 93.9 mm
- board text removed: "+"
- board text removed: "3"
- board text removed: ":"
- board text removed: "Diodes 󰱫"
- board text removed: "Keys"
- board text removed: "Made wi"
- board text removed: "Made with  by"
- board text removed: "Rever"
- board text removed: "manni"
- board text removed: "sible 󰌌"
- board text removed: "th  by manni"
- board text removed: "󰬽"
- board text removed: "󰭁"
