File: PCB/RELIC.kicad_sch (KiCad schematic)
At the start: 82 parts, among them J1 Conn_01x02, J2 Conn_01x02, SW1 SW_Push_45deg, SW10 SW_Push_45deg, SW11 SW_Push_45deg, SW12 SW_Push_45deg, SW13 SW_Push_45deg, SW14 SW_Push_45deg, SW15 SW_Push_45deg, SW16 SW_Push_45deg, SW17 SW_Push_45deg, SW18 SW_Push_45deg, SW19 SW_Push_45deg, SW2 SW_Push_45deg, SW20 SW_Push_45deg, SW21 SW_Push_45deg, SW22 SW_Push_45deg, SW23 SW_Push_45deg, SW24 SW_Push_45deg, SW25 SW_Push_45deg, SW26 SW_Push_45deg, SW27 SW_Push_45deg, SW28 SW_Push_45deg, SW29 SW_Push_45deg, SW3 SW_Push_45deg, SW30 SW_Push_45deg, SW31 SW_Push_45deg, SW32 SW_Push_45deg, SW33 SW_Push_45deg, SW34 SW_Push_45deg, SW35 SW_Push_45deg, SW36 SW_Push_45deg, SW37 SW_Push_45deg, SW38 SW_Push_45deg, SW39 SW_SPDT, SW4 SW_Push_45deg, SW40 SW_SPDT, SW5 SW_Push_45deg, SW6 SW_Push_45deg, SW7 SW_Push_45deg, SW8 SW_Push_45deg, SW9 SW_Push_45deg, U1 Seeeduino Xiao nRF52840, U2 Seeeduino Xiao nRF52840

Commit message: Rename stuff
Parts:
- removed D19, D38: D, Diode_SMD:D_SOD-123, symbol Device:D
- removed SW19, SW38: SW_Push_45deg, MX_Hotswap:MX-Hotswap-1U, symbol Switch:SW_Push_45deg
- D1, D10, D11, D12, D13, D14, D15, D16, D17, D18, D2, D20, D21, D22, D23, D24, D25, D26, D27, D28, D29, D3, D30, D31, D32, D33, D34, D35, D36, D37, D4, D5, D6, D7, D8, D9: footprint Diode_SMD:D_SOD-123 -> ScottoKeebs_Components:Diode_DO-35
Connections:
- net GNDR is gone; now on net GNDL: U2.22 (GND)
- net R1R is gone; now on net R1L: U2.12 (P1.14)
- net R2R is gone; now on net R2L: U2.13 (P1.13)
- net R3R is gone; now on net R3L: U2.14 (P1.12)
- net C0: no longer SW12.1
- net C0L: now also SW35.1; no longer SW31.1
- net C1: now also SW12.1; no longer SW13.1
- net C1L: now also SW31.1, SW36.1; no longer SW32.1
- net C2: now also SW13.1, SW16.1; no longer SW14.1, SW17.1
- net C2L: now also SW32.1, SW37.1; no longer SW33.1, SW36.1
- net C3: now also SW14.1, SW17.1; no longer SW15.1, SW18.1
- net C3L: now also SW33.1; no longer SW34.1, SW37.1
- net C4: now also SW15.1, SW18.1; no longer SW16.1
- net C4L: now also SW34.1; no longer SW35.1
- net R2: no longer D16.1 (K)
- net R2L: no longer D35.1 (K)
- net R3: now also D16.1 (K)
- net R3L: now also D35.1 (K)
Other:
- moved on the sheet: D1, D10, D16, D2, D20, D21, D22, D23, D24, D25, D26, D27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
