File: PCB/RELIC.kicad_pcb (KiCad board)
At the start: 2 copper layers, 246.4 x 128.5 mm, 84 parts, among them J1 Conn_01x02, J2 Conn_01x02, SW1 SW_Push_45deg, SW10 SW_Push_45deg, SW11 SW_Push_45deg, SW12 SW_Push_45deg, SW13 SW_Push_45deg, SW14 SW_Push_45deg, SW15 SW_Push_45deg, SW16 SW_Push_45deg, SW17 SW_Push_45deg, SW18 SW_Push_45deg, SW2 SW_Push_45deg, SW20 SW_Push_45deg, SW21 SW_Push_45deg, SW22 SW_Push_45deg, SW23 SW_Push_45deg, SW24 SW_Push_45deg, SW25 SW_Push_45deg, SW26 SW_Push_45deg, SW27 SW_Push_45deg, SW28 SW_Push_45deg, SW29 SW_Push_45deg, SW3 SW_Push_45deg, SW30 SW_Push_45deg, SW31 SW_Push_45deg, SW32 SW_Push_45deg, SW33 SW_Push_45deg, SW34 SW_Push_45deg, SW35 SW_Push_45deg, SW36 SW_Push_45deg, SW37 SW_Push_45deg, SW39 SW_SPDT, SW4 SW_Push_45deg, SW40 SW_SPDT, SW5 SW_Push_45deg, SW6 SW_Push_45deg, SW7 SW_Push_45deg, SW8 SW_Push_45deg, SW9 SW_Push_45deg, U1 Seeeduino Xiao nRF52840, U2 Seeeduino Xiao nRF52840

Commit message: meow
Parts:
- moved REF** 2.00 mm to (70.5, 41.2), turned to -90 degrees
Changed lines of the file:
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@@
 		(allow_soldermask_bridges_in_footprints no)
 		(tenting front back)
-		(grid_origin 248.431298 161.433964)
+		(grid_origin 67.5333 39.193964)
 		(pcbplotparams
-			(layerselection 0x00000000_00000000_55555555_75555550)
+			(layerselection 0x00000000_00000000_55555555_555f5550)
 			(plot_on_all_layers_selection 0x00000000_00000000_00000000_00000000)
 			(disableapertmacros no)
@@
 			(drillshape 0)
 			(scaleselection 1)
-			(outputdirectory "/home/manni/Downloads/")
+			(outputdirectory "/home/manni/Desktop/")
 		)
 	)
@@
 	(footprint "PCM_marbastlib-various:mousebites_2mm"
 		(layer "F.Cu")
-		(at 70.521298 39.193964 90)
+		(at 70.521298 41.193964 -90)
 		(property "Reference" "REF**"
 			(at -4 -2.75 90)
@@
 		(attr exclude_from_pos_files exclude_from_bom)
 		(fp_arc
-			(start 0 -3)
-			(mid -1 -2)
-			(end -2 -3)
+			(start -2 3)
+			(mid -1 2)
+			(end 0 3)
 			(stroke
 				(width 0.05)
@@
 		)
 		(fp_arc
-			(start -2 3)
-			(mid -1 2)
-			(end 0 3)
+			(start 0 -3)
+			(mid -1 -2)
+			(end -2 -3)
 			(stroke
 				(width 0.05)
@@
 		)
 		(pad "" np_thru_hole circle
-			(at 0.05 -1.85 90)
+			(at 0.05 -1.85 270)
 			(size 0.5 0.5)
 			(drill 0.5)
@@
 		)
 		(pad "" np_thru_hole circle
-			(at 0.05 -1.11 90)
+			(at 0.05 -1.11 270)
 			(size 0.5 0.5)
 			(drill 0.5)
@@
 		)
 		(pad "" np_thru_hole circle
-			(at 0.05 -0.37 90)
+			(at 0.05 -0.37 270)
 			(size 0.5 0.5)
 			(drill 0.5)
@@
 		)
 		(pad "" np_thru_hole circle
-			(at 0.05 0.37 90)
+			(at 0.05 0.37 270)
 			(size 0.5 0.5)
 			(drill 0.5)
@@
 		)
 		(pad "" np_thru_hole circle
-			(at 0.05 1.11 90)
+			(at 0.05 1.11 270)
 			(size 0.5 0.5)
 			(drill 0.5)
@@
 		)
 		(pad "" np_thru_hole circle
-			(at 0.05 1.85 90)
+			(at 0.05 1.85 270)
 			(size 0.5 0.5)
 			(drill 0.5)
@@
 	)
 	(segment
-		(start 139.761298 95.676464)
-		(end 132.361298 88.276464)
-		(width 0.2)
-		(layer "F.Cu")
-		(net 60)
-	)
-	(segment
-		(start 129.247296 71.042964)
-		(end 127.696297 71.042964)
+		(start 132.361298 88.276464)
+		(end 132.361298 83.640466)
 		(width 0.2)
 		(layer "F.Cu")
@@
 	)
 	(segment
-		(start 132.361298 83.640466)
-		(end 129.247296 80.526464)
+		(start 129.247296 80.526464)
+		(end 129.247296 70.113964)
 		(width 0.2)
 		(layer "F.Cu")
@@
 	)
 	(segment
-		(start 127.696297 71.042964)
+		(start 129.247296 70.113964)
 		(end 127.696297 70.113964)
 		(width 0.2)
@@
 	)
 	(segment
-		(start 129.247296 80.526464)
-		(end 129.247296 71.042964)
+		(start 139.761298 95.676464)
+		(end 132.361298 88.276464)
 		(width 0.2)
 		(layer "F.Cu")
@@
 	)
 	(segment
-		(start 132.361298 88.276464)
-		(end 132.361298 83.640466)
+		(start 132.361298 83.640466)
+		(end 129.247296 80.526464)
 		(width 0.2)
 		(layer "F.Cu")
